File: Schematics/Schematics.kicad_sch (KiCad schematic)
At the start: 8 parts, among them Q1 BC547, U1 CY8C5888LTI-LP09, U2 LM78L05, U3 Adafruit_BNO08x

Commit message: TILFØJEDE LIDT PINS
Parts:
- Q1: footprint (none) -> Package_TO_SOT_THT:TO-92
- R1: footprint (none) -> Resistor_THT:R_Axial_DIN0204_L3.6mm_D1.6mm_P7.62mm_Horizontal
- U1: footprint Package_QFP:TQFP-64_14x14mm_P0.8mm -> Module:MODULE_CY8CKIT-059 PSOC5
- U3: footprint (none) -> Module:Adafruit_BNO08x home made
Connections:
- net +5V: now also U1.J1.1 (VDD); no longer U1. (RES)
- net Buzzer: now also U1.J2.1 (P2.0); no longer U1. (RES)
- net GND: now also U1.J1.2 (GND), U1.J1.26 (GND), U1.J2.25 (GND); no longer U1. (RES)
- net I2C_SCL: now also U1.J2.16 (P12.0/SCL); no longer U1. (RES)
- net I2C_SDA: now also U1.J2.15 (P12.1/SDA); no longer U1. (RES)
- net Reset NANO: now also U1.J2.4 (P2.3); no longer U1. (RES)
Changed lines of the file:
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@@
 			)
 		)
-		(property "Footprint" "Package_QFP:TQFP-64_14x14mm_P0.8mm"
+		(property "Footprint" "Module:MODULE_CY8CKIT-059 PSOC5"
 			(at 187.96 139.7 0)
 			(effects
@@
 		(pin ""
 		)
-		(pin ""
-		)
-		(pin ""
-		)
-		(pin ""
-		)
-		(pin ""
-		)
-		(pin ""
-		)
-		(pin ""
-		)
-		(pin ""
-		)
-		(pin ""
-		)
-		(pin ""
-		)
-		(pin ""
-		)
-		(pin ""
-		)
-		(pin ""
-		)
-		(pin ""
-		)
-		(pin ""
-		)
-		(pin ""
-		)
-		(pin ""
-		)
-		(pin ""
-		)
-		(pin ""
-		)
-		(pin ""
-		)
-		(pin ""
-		)
-		(pin ""
-		)
-		(pin ""
-		)
-		(pin ""
-		)
-		(pin ""
-		)
-		(pin ""
-		)
-		(pin ""
-		)
-		(pin ""
-		)
-		(pin ""
-		)
-		(pin ""
-		)
-		(pin ""
-		)
-		(pin ""
-		)
-		(pin ""
-		)
-		(pin ""
-		)
-		(pin ""
+		(pin "J2.26"
+		)
+		(pin ""
+		)
+		(pin "J2.4"
+		)
+		(pin ""
+		)
+		(pin "J2.16"
+		)
+		(pin ""
+		)
+		(pin "J2.25"
+		)
+		(pin ""
+		)
+		(pin "J2.15"
+		)
+		(pin "J1.1"
+		)
+		(pin ""
+		)
+		(pin ""
+		)
+		(pin ""
+		)
+		(pin ""
+		)
+		(pin ""
+		)
+		(pin ""
+		)
+		(pin ""
+		)
+		(pin "J1.2"
+		)
+		(pin ""
+		)
+		(pin "J1.24"
+		)
+		(pin ""
+		)
+		(pin "J1.26"
+		)
+		(pin "J1.23"
+		)
+		(pin "J1.22"
+		)
+		(pin "J2.1"
+		)
+		(pin ""
+		)
+		(pin ""
+		)
+		(pin ""
+		)
+		(pin ""
+		)
+		(pin ""
+		)
+		(pin ""
+		)
+		(pin ""
+		)
+		(pin ""
+		)
+		(pin "J1.25"
 		)
 		(pin ""
@@
 			)
 		)
-		(property "Footprint" ""
+		(property "Footprint" "Module:Adafruit_BNO08x home made"
 			(at 90.17 110.49 0)
 			(effects
@@
 			)
 		)
-		(property "Footprint" ""
+		(property "Footprint" "Resistor_THT:R_Axial_DIN0204_L3.6mm_D1.6mm_P7.62mm_Horizontal"
 			(at 54.61 47.498 90)
 			(effects
@@
 			)
 		)
-		(property "Footprint" ""
+		(property "Footprint" "Package_TO_SOT_THT:TO-92"
 			(at 7.62 45.72 0)
 			(effects

Commit message: opdaterede schematics
Parts:
- added D1, D2: LED, symbol Device:LED
- added M1: Feedback Servo, symbol Motor:Motor_Servo
- added R2, R3: 220, symbol Device:R
- added SW1: RotaryEncoder_Switch, symbol Device:RotaryEncoder_Switch
Connections:
- net +5V: now also M1.2 (+)
- net GND: now also M1.3 (-), R2.2, R3.2, SW1.C, SW1.S1
- net Servo_PWM: now reaches U1. (RES)
- net Servo_PWM: now also M1.1 (PWM)
- new net: D2.1 (K), R3.1
- new net: D1.1 (K), R2.1
- new net Butt: SW1.S2, U1. (RES)
- new net Green_LED: D2.2 (A), U1. (RES)
- new net Red_LED: D1.2 (A), U1. (RES)
- new net Rot_A: SW1.A, U1. (RES)
- new net Rot_B: SW1.B, U1. (RES)
- new net Servo_FB: M1. (FB), U1. (RES)
Other:
- note added: "Servo"
- note added: "UI"
- moved on the sheet: U3
